Commit message: Point URDF to correct sub-meshes.

File: robot/man1.urdf (robot description, URDF)
Before this commit: robot man1, 64 links, 63 joints
Links:
- link Chest: geometry collision mesh filename=package://libhuman/robot/mesh/Chest_mesh.dae scale=1 1 1; visual mesh filename=package://libhuman/robot/mesh/Chest_mesh.dae scale=1 1 1
- link Head: geometry collision mesh filename=package://libhuman/robot/mesh/Head_mesh.dae scale=1 1 1; visual mesh filename=package://libhuman/robot/mesh/Head_mesh.dae scale=1 1 1
- link Hips: geometry collision mesh filename=package://libhuman/robot/mesh/Hips_mesh.dae scale=1 1 1; visual mesh filename=package://libhuman/robot/mesh/Hips_mesh.dae scale=1 1 1
- link LCalf: geometry collision mesh filename=package://libhuman/robot/mesh/LCalf_mesh.dae scale=1 1 1; visual mesh filename=package://libhuman/robot/mesh/LCalf_mesh.dae scale=1 1 1
- link LCollar: geometry collision mesh filename=package://libhuman/robot/mesh/LCollar_mesh.dae scale=1 1 1; visual mesh filename=package://libhuman/robot/mesh/LCollar_mesh.dae scale=1 1 1
- link LFing10: geometry collision mesh filename=package://libhuman/robot/mesh/LFing10_mesh.dae scale=1 1 1; visual mesh filename=package://libhuman/robot/mesh/LFing10_mesh.dae scale=1 1 1
- link LFing11: geometry collision mesh filename=package://libhuman/robot/mesh/LFing11_mesh.dae scale=1 1 1; visual mesh filename=package://libhuman/robot/mesh/LFing11_mesh.dae scale=1 1 1
- link LFing12: geometry collision mesh filename=package://libhuman/robot/mesh/LFing12_mesh.dae scale=1 1 1; visual mesh filename=package://libhuman/robot/mesh/LFing12_mesh.dae scale=1 1 1
- link LFing20: geometry collision mesh filename=package://libhuman/robot/mesh/LFing20_mesh.dae scale=1 1 1; visual mesh filename=package://libhuman/robot/mesh/LFing20_mesh.dae scale=1 1 1
- link LFing21: geometry collision mesh filename=package://libhuman/robot/mesh/LFing21_mesh.dae scale=1 1 1; visual mesh filename=package://libhuman/robot/mesh/LFing21_mesh.dae scale=1 1 1
- link LFing22: geometry collision mesh filename=package://libhuman/robot/mesh/LFing22_mesh.dae scale=1 1 1; visual mesh filename=package://libhuman/robot/mesh/LFing22_mesh.dae scale=1 1 1
- link LFing30: geometry collision mesh filename=package://libhuman/robot/mesh/LFing30_mesh.dae scale=1 1 1; visual mesh filename=package://libhuman/robot/mesh/LFing30_mesh.dae scale=1 1 1
- link LFing31: geometry collision mesh filename=package://libhuman/robot/mesh/LFing31_mesh.dae scale=1 1 1; visual mesh filename=package://libhuman/robot/mesh/LFing31_mesh.dae scale=1 1 1
- link LFing32: geometry collision mesh filename=package://libhuman/robot/mesh/LFing32_mesh.dae scale=1 1 1; visual mesh filename=package://libhuman/robot/mesh/LFing32_mesh.dae scale=1 1 1
- link LFing40: geometry collision mesh filename=package://libhuman/robot/mesh/LFing40_mesh.dae scale=1 1 1; visual mesh filename=package://libhuman/robot/mesh/LFing40_mesh.dae scale=1 1 1
- link LFing41: geometry collision mesh filename=package://libhuman/robot/mesh/LFing41_mesh.dae scale=1 1 1; visual mesh filename=package://libhuman/robot/mesh/LFing41_mesh.dae scale=1 1 1
- link LFing42: geometry collision mesh filename=package://libhuman/robot/mesh/LFing42_mesh.dae scale=1 1 1; visual mesh filename=package://libhuman/robot/mesh/LFing42_mesh.dae scale=1 1 1
- link LFoot: geometry collision mesh filename=package://libhuman/robot/mesh/LFoot_mesh.dae scale=1 1 1; visual mesh filename=package://libhuman/robot/mesh/LFoot_mesh.dae scale=1 1 1
- link LForearm: geometry collision mesh filename=package://libhuman/robot/mesh/LForearm_mesh.dae scale=1 1 1; visual mesh filename=package://libhuman/robot/mesh/LForearm_mesh.dae scale=1 1 1
- link LHand: geometry collision mesh filename=package://libhuman/robot/mesh/LHand_mesh.dae scale=1 1 1; visual mesh filename=package://libhuman/robot/mesh/LHand_mesh.dae scale=1 1 1
- link LHand2: geometry collision mesh filename=package://libhuman/robot/mesh/LHand2_mesh.dae scale=1 1 1; visual mesh filename=package://libhuman/robot/mesh/LHand2_mesh.dae scale=1 1 1
- link LHand3: geometry collision mesh filename=package://libhuman/robot/mesh/LHand3_mesh.dae scale=1 1 1; visual mesh filename=package://libhuman/robot/mesh/LHand3_mesh.dae scale=1 1 1
- link LShoulder: geometry collision mesh filename=package://libhuman/robot/mesh/LShoulder_mesh.dae scale=1 1 1; visual mesh filename=package://libhuman/robot/mesh/LShoulder_mesh.dae scale=1 1 1
- link LShoulder2: geometry collision mesh filename=package://libhuman/robot/mesh/LShoulder2_mesh.dae scale=1 1 1; visual mesh filename=package://libhuman/robot/mesh/LShoulder2_mesh.dae scale=1 1 1
- link LShoulder3: geometry collision mesh filename=package://libhuman/robot/mesh/LShoulder3_mesh.dae scale=1 1 1; visual mesh filename=package://libhuman/robot/mesh/LShoulder3_mesh.dae scale=1 1 1
- link LThigh: geometry collision mesh filename=package://libhuman/robot/mesh/LThigh_mesh.dae scale=1 1 1; visual mesh filename=package://libhuman/robot/mesh/LThigh_mesh.dae scale=1 1 1
- link LThumb0: geometry collision mesh filename=package://libhuman/robot/mesh/LThumb0_mesh.dae scale=1 1 1; visual mesh filename=package://libhuman/robot/mesh/LThumb0_mesh.dae scale=1 1 1
- link LThumb1: geometry collision mesh filename=package://libhuman/robot/mesh/LThumb1_mesh.dae scale=1 1 1; visual mesh filename=package://libhuman/robot/mesh/LThumb1_mesh.dae scale=1 1 1
- link LThumb2: geometry collision mesh filename=package://libhuman/robot/mesh/LThumb2_mesh.dae scale=1 1 1; visual mesh filename=package://libhuman/robot/mesh/LThumb2_mesh.dae scale=1 1 1
- link LThumbBase: geometry collision mesh filename=package://libhuman/robot/mesh/LThumbBase_mesh.dae scale=1 1 1; visual mesh filename=package://libhuman/robot/mesh/LThumbBase_mesh.dae scale=1 1 1
- link LThumbBase2: geometry collision mesh filename=package://libhuman/robot/mesh/LThumbBase2_mesh.dae scale=1 1 1; visual mesh filename=package://libhuman/robot/mesh/LThumbBase2_mesh.dae scale=1 1 1
- link LToe: geometry collision mesh filename=package://libhuman/robot/mesh/LToe_mesh.dae scale=1 1 1; visual mesh filename=package://libhuman/robot/mesh/LToe_mesh.dae scale=1 1 1
- link LeftEye: geometry collision mesh filename=package://libhuman/robot/mesh/LeftEye_mesh.dae scale=1 1 1; visual mesh filename=package://libhuman/robot/mesh/LeftEye_mesh.dae scale=1 1 1
- link Neck: geometry collision mesh filename=package://libhuman/robot/mesh/Neck_mesh.dae scale=1 1 1; visual mesh filename=package://libhuman/robot/mesh/Neck_mesh.dae scale=1 1 1
- link RCalf: geometry collision mesh filename=package://libhuman/robot/mesh/RCalf_mesh.dae scale=1 1 1; visual mesh filename=package://libhuman/robot/mesh/RCalf_mesh.dae scale=1 1 1
- link RCollar: geometry collision mesh filename=package://libhuman/robot/mesh/RCollar_mesh.dae scale=1 1 1; visual mesh filename=package://libhuman/robot/mesh/RCollar_mesh.dae scale=1 1 1
- link RFing10: geometry collision mesh filename=package://libhuman/robot/mesh/RFing10_mesh.dae scale=1 1 1; visual mesh filename=package://libhuman/robot/mesh/RFing10_mesh.dae scale=1 1 1
- link RFing11: geometry collision mesh filename=package://libhuman/robot/mesh/RFing11_mesh.dae scale=1 1 1; visual mesh filename=package://libhuman/robot/mesh/RFing11_mesh.dae scale=1 1 1
- link RFing12: geometry collision mesh filename=package://libhuman/robot/mesh/RFing12_mesh.dae scale=1 1 1; visual mesh filename=package://libhuman/robot/mesh/RFing12_mesh.dae scale=1 1 1
- link RFing20: geometry collision mesh filename=package://libhuman/robot/mesh/RFing20_mesh.dae scale=1 1 1; visual mesh filename=package://libhuman/robot/mesh/RFing20_mesh.dae scale=1 1 1
- link RFing21: geometry collision mesh filename=package://libhuman/robot/mesh/RFing21_mesh.dae scale=1 1 1; visual mesh filename=package://libhuman/robot/mesh/RFing21_mesh.dae scale=1 1 1
- link RFing22: geometry collision mesh filename=package://libhuman/robot/mesh/RFing22_mesh.dae scale=1 1 1; visual mesh filename=package://libhuman/robot/mesh/RFing22_mesh.dae scale=1 1 1
- link RFing30: geometry collision mesh filename=package://libhuman/robot/mesh/RFing30_mesh.dae scale=1 1 1; visual mesh filename=package://libhuman/robot/mesh/RFing30_mesh.dae scale=1 1 1
- link RFing31: geometry collision mesh filename=package://libhuman/robot/mesh/RFing31_mesh.dae scale=1 1 1; visual mesh filename=package://libhuman/robot/mesh/RFing31_mesh.dae scale=1 1 1
- link RFing32: geometry collision mesh filename=package://libhuman/robot/mesh/RFing32_mesh.dae scale=1 1 1; visual mesh filename=package://libhuman/robot/mesh/RFing32_mesh.dae scale=1 1 1
- link RFing40: geometry collision mesh filename=package://libhuman/robot/mesh/RFing40_mesh.dae scale=1 1 1; visual mesh filename=package://libhuman/robot/mesh/RFing40_mesh.dae scale=1 1 1
- link RFing41: geometry collision mesh filename=package://libhuman/robot/mesh/RFing41_mesh.dae scale=1 1 1; visual mesh filename=package://libhuman/robot/mesh/RFing41_mesh.dae scale=1 1 1
- link RFing42: geometry collision mesh filename=package://libhuman/robot/mesh/RFing42_mesh.dae scale=1 1 1; visual mesh filename=package://libhuman/robot/mesh/RFing42_mesh.dae scale=1 1 1
- link RFoot: geometry collision mesh filename=package://libhuman/robot/mesh/RFoot_mesh.dae scale=1 1 1; visual mesh filename=package://libhuman/robot/mesh/RFoot_mesh.dae scale=1 1 1
- link RForearm: geometry collision mesh filename=package://libhuman/robot/mesh/RForearm_mesh.dae scale=1 1 1; visual mesh filename=package://libhuman/robot/mesh/RForearm_mesh.dae scale=1 1 1
- link RHand: geometry collision mesh filename=package://libhuman/robot/mesh/RHand_mesh.dae scale=1 1 1; visual mesh filename=package://libhuman/robot/mesh/RHand_mesh.dae scale=1 1 1
- link RHand2: geometry collision mesh filename=package://libhuman/robot/mesh/RHand2_mesh.dae scale=1 1 1; visual mesh filename=package://libhuman/robot/mesh/RHand2_mesh.dae scale=1 1 1
- link RHand3: geometry collision mesh filename=package://libhuman/robot/mesh/RHand3_mesh.dae scale=1 1 1; visual mesh filename=package://libhuman/robot/mesh/RHand3_mesh.dae scale=1 1 1
- link RShoulder: geometry collision mesh filename=package://libhuman/robot/mesh/RShoulder_mesh.dae scale=1 1 1; visual mesh filename=package://libhuman/robot/mesh/RShoulder_mesh.dae scale=1 1 1
- link RShoulder2: geometry collision mesh filename=package://libhuman/robot/mesh/RShoulder2_mesh.dae scale=1 1 1; visual mesh filename=package://libhuman/robot/mesh/RShoulder2_mesh.dae scale=1 1 1
- link RShoulder3: geometry collision mesh filename=package://libhuman/robot/mesh/RShoulder3_mesh.dae scale=1 1 1; visual mesh filename=package://libhuman/robot/mesh/RShoulder3_mesh.dae scale=1 1 1
- link RThigh: geometry collision mesh filename=package://libhuman/robot/mesh/RThigh_mesh.dae scale=1 1 1; visual mesh filename=package://libhuman/robot/mesh/RThigh_mesh.dae scale=1 1 1
- link RThumb0: geometry collision mesh filename=package://libhuman/robot/mesh/RThumb0_mesh.dae scale=1 1 1; visual mesh filename=package://libhuman/robot/mesh/RThumb0_mesh.dae scale=1 1 1
- link RThumb1: geometry collision mesh filename=package://libhuman/robot/mesh/RThumb1_mesh.dae scale=1 1 1; visual mesh filename=package://libhuman/robot/mesh/RThumb1_mesh.dae scale=1 1 1
- link RThumb2: geometry collision mesh filename=package://libhuman/robot/mesh/RThumb2_mesh.dae scale=1 1 1; visual mesh filename=package://libhuman/robot/mesh/RThumb2_mesh.dae scale=1 1 1
- link RThumbBase: geometry collision mesh filename=package://libhuman/robot/mesh/RThumbBase_mesh.dae scale=1 1 1; visual mesh filename=package://libhuman/robot/mesh/RThumbBase_mesh.dae scale=1 1 1
- link RThumbBase2: geometry collision mesh filename=package://libhuman/robot/mesh/RThumbBase2_mesh.dae scale=1 1 1; visual mesh filename=package://libhuman/robot/mesh/RThumbBase2_mesh.dae scale=1 1 1
- link RToe: geometry collision mesh filename=package://libhuman/robot/mesh/RToe_mesh.dae scale=1 1 1; visual mesh filename=package://libhuman/robot/mesh/RToe_mesh.dae scale=1 1 1
- link RightEye: geometry collision mesh filename=package://libhuman/robot/mesh/RightEye_mesh.dae scale=1 1 1; visual mesh filename=package://libhuman/robot/mesh/RightEye_mesh.dae scale=1 1 1
